File: Peapod PCB.sch (KiCad schematic (older format))
At the start: 18 parts, among them J1 CONN_01X01, J2 CONN_01X02, J3 CONN_01X06, J4 CONN_01X01, J5 CONN_01X01, J6 CONN_01X01, J7 CONN_01X02, J8 CONN_01X01, U1 ESP8266

Commit message: Updated logo, year, names
Parts:
- BT1: symbol Battery_Cell -> Peapod-PCB-rescue:Battery_Cell
- BTN1, BTN2, BTN3: symbol Pushbutton -> pushbutton:Pushbutton
- J1, J4, J5, J6, J8: symbol CONN_01X01 -> Peapod-PCB-rescue:CONN_01X01
- J2, J7: symbol CONN_01X02 -> Peapod-PCB-rescue:CONN_01X02
- J3: symbol CONN_01X06 -> Peapod-PCB-rescue:CONN_01X06
- R1, R2, R3, R4, R5: symbol R -> Peapod-PCB-rescue:R
- U1: symbol ESP8266 -> esp8266:ESP8266
Connections:
- wire segments 46 -> 45
Changed lines of the file:
@@
-EESchema Schematic File Version 2
-LIBS:Peapod PCB-rescue
-LIBS:power
-LIBS:device
-LIBS:transistors
-LIBS:conn
-LIBS:linear
-LIBS:regul
-LIBS:74xx
-LIBS:cmos4000
-LIBS:adc-dac
-LIBS:memory
-LIBS:xilinx
-LIBS:microcontrollers
-LIBS:dsp
-LIBS:microchip
-LIBS:analog_switches
-LIBS:motorola
-LIBS:texas
-LIBS:intel
-LIBS:audio
-LIBS:interface
-LIBS:digital-audio
-LIBS:philips
-LIBS:display
-LIBS:cypress
-LIBS:siliconi
-LIBS:opto
-LIBS:atmel
-LIBS:contrib
-LIBS:valves
-LIBS:esp8266
-LIBS:pushbutton
+EESchema Schematic File Version 4
 LIBS:Peapod PCB-cache
-EELAYER 25 0
+EELAYER 26 0
 EELAYER END
 $Descr A4 11693 8268
@@
 $EndDescr
 $Comp
-L Battery_Cell BT1
+L Peapod-PCB-rescue:Battery_Cell BT1
 U 1 1 599321E0
 P 4950 4125
@@
 $EndComp
 $Comp
-L GND #PWR2
+L power:GND #PWR2
 U 1 1 59932223
 P 4850 4225
@@
 $EndComp
 $Comp
-L GND #PWR8
+L power:GND #PWR8
 U 1 1 59932907
 P 6800 4100
@@
 $EndComp
 $Comp
-L GND #PWR1
+L power:GND #PWR1
 U 1 1 5993357D
 P 4500 3825
@@
 $EndComp
 $Comp
-L CONN_01X01 J5
+L Peapod-PCB-rescue:CONN_01X01 J5
 U 1 1 59933C1C
 P 7450 3175
@@
 $EndComp
 $Comp
-L CONN_01X01 J6
+L Peapod-PCB-rescue:CONN_01X01 J6
 U 1 1 59933C73
 P 7450 3325
@@
 $EndComp
 $Comp
-L CONN_01X01 J1
+L Peapod-PCB-rescue:CONN_01X01 J1
 U 1 1 59933CDE
 P 4525 3275
@@
 $EndComp
 $Comp
-L +3.3V #PWR5
+L power:+3.3V #PWR5
 U 1 1 59933FE4
 P 5300 3175
@@
 $EndComp
 $Comp
-L +3.3V #PWR4
+L power:+3.3V #PWR4
 U 1 1 59934256
 P 4950 3925
@@
 $EndComp
 $Comp
-L R R1
+L Peapod-PCB-rescue:R R1
 U 1 1 59934609
 P 4675 3025
@@
 	4875 3025 5325 3025
 $Comp
-L R R2
+L Peapod-PCB-rescue:R R2
 U 1 1 59934849
 P 4875 2750
@@
 Connection ~ 4875 3025
 $Comp
-L CONN_01X02 J7
+L Peapod-PCB-rescue:CONN_01X02 J7
 U 1 1 5993514F
 P 7450 3600
@@
 	7250 3750 7250 3650
 $Comp
-L R R4
+L Peapod-PCB-rescue:R R4
 U 1 1 59935339
 P 7100 3625
@@
 Connection ~ 7100 3475
 $Comp
-L CONN_01X02 J2
+L Peapod-PCB-rescue:CONN_01X02 J2
 U 1 1 5993627D
 P 5175 2500
@@
 $EndComp
 $Comp
-L GND #PWR6
+L power:GND #PWR6
 U 1 1 599363AF
 P 5325 2700
@@
 $EndComp
 $Comp
-L +3.3V #PWR12
+L power:+3.3V #PWR12
 U 1 1 599466C8
 P 7100 3875
@@
 	7100 3775 7100 3875
 $Comp
-L R R3
+L Peapod-PCB-rescue:R R3
 U 1 1 59946DA6
 P 6825 3625
@@
 $EndComp
 $Comp
-L R R5
+L Peapod-PCB-rescue:R R5
 U 1 1 59946FC4
 P 6800 3925
@@
 	6625 3775 6800 3775
 $Comp
-L +3.3V #PWR11
+L power:+3.3V #PWR11
 U 1 1 59948486
 P 6975 3700
@@
 	4875 2900 4875 3025
 $Comp
-L GND #PWR3
+L power:GND #PWR3
 U 1 1 5994872F
 P 4875 2525
@@
 	4875 2525 4875 2600
 $Comp
-L GND #PWR13
+L power:GND #PWR13
 U 1 1 599488CC
 P 7250 3750
@@
 $EndComp
 $Comp
-L GND #PWR7
+L power:GND #PWR7
 U 1 1 59948924
 P 6625 4000
@@
 	4525 3025 4525 3075
 $Comp
-L ESP8266 U1
+L esp8266:ESP8266 U1
 U 1 1 59932095
 P 5925 3275
@@
 	5325 3925 4950 3925
 $Comp
-L CONN_01X06 J3
+L Peapod-PCB-rescue:CONN_01X06 J3
 U 1 1 59947FD8
 P 7500 2450
@@
 $EndComp
 $Comp
-L GND #PWR10
+L power:GND #PWR10
 U 1 1 599480D5
 P 6875 2200
@@
 	6875 2200 7300 2200
 $Comp
-L +3.3V #PWR9
+L power:+3.3V #PWR9
 U 1 1 599481A2
 P 6850 2400
@@
 	6800 2875 6800 2600
 Wire Wire Line
-	6800 2600 6800 2600
-Wire Wire Line
 	6800 2600 7300 2600
 Wire Wire Line
@@
 NoConn ~ 7300 2300
 $Comp
-L Pushbutton BTN2
+L pushbutton:Pushbutton BTN2
 U 1 1 5994A123
 P 5150 3475
@@
 $EndComp
 $Comp
-L Pushbutton BTN1
+L pushbutton:Pushbutton BTN1
 U 1 1 5994A192
 P 4775 3625
@@
 $EndComp
 $Comp
-L Pushbutton BTN3
+L pushbutton:Pushbutton BTN3
 U 1 1 5994A1EB
 P 5150 3775
@@
 $EndComp
 $Comp
-L CONN_01X01 J4
+L Peapod-PCB-rescue:CONN_01X01 J4
 U 1 1 5995C3B2
 P 5825 2100
@@
 $EndComp
 $Comp
-L CONN_01X01 J8
+L Peapod-PCB-rescue:CONN_01X01 J8
 U 1 1 5995C3FF
 P 6375 2100
